File: hw/mows.sch (KiCad schematic (older format))
At the start: 18 parts, among them J1 ICSP, J2 STX882, J3 DHT22, J4 WSPD, J5 WDIR, J6 RAIN, U1 MCP1700-3302E_TO92, U2 ATTINY85-20PU

Commit message: ctimer support for different clocks
Parts:
- D1: symbol D_Schottky -> mows-rescue:D_Schottky
- J1: symbol Conn_01x06 -> mows-rescue:Conn_01x06
- J2, J3: symbol Conn_01x03 -> mows-rescue:Conn_01x03
- J4, J5, J6, con_bat1, con_sun1: symbol Conn_01x02 -> mows-rescue:Conn_01x02
- R1, R2, R3, R4, R5, R6, R7: symbol R -> mows-rescue:R
- U1: symbol MCP1700-3302E_TO92 -> mows-rescue:MCP1700-3302E_TO92
- U2: symbol ATTINY85-20PU -> mows-rescue:ATTINY85-20PU
Connections:
- net labels removed: SUN
- wire segments 60 -> 61
Changed lines of the file:
@@
-EESchema Schematic File Version 2
-LIBS:power
-LIBS:device
-LIBS:transistors
-LIBS:conn
-LIBS:linear
-LIBS:regul
-LIBS:74xx
-LIBS:cmos4000
-LIBS:adc-dac
-LIBS:memory
-LIBS:xilinx
-LIBS:microcontrollers
-LIBS:dsp
-LIBS:microchip
-LIBS:analog_switches
-LIBS:motorola
-LIBS:texas
-LIBS:intel
-LIBS:audio
-LIBS:interface
-LIBS:digital-audio
-LIBS:philips
-LIBS:display
-LIBS:cypress
-LIBS:siliconi
-LIBS:opto
-LIBS:atmel
-LIBS:contrib
-LIBS:valves
+EESchema Schematic File Version 4
 LIBS:mows-cache
-EELAYER 25 0
+EELAYER 26 0
 EELAYER END
 $Descr A4 11693 8268
@@
 $EndDescr
 $Comp
-L ATTINY85-20PU U2
+L mows-rescue:ATTINY85-20PU U2
 U 1 1 594FB4D7
 P 3100 2650
@@
 $EndComp
 $Comp
-L R R4
+L mows-rescue:R R4
 U 1 1 594FB5E0
 P 5050 1450
@@
 $EndComp
 $Comp
-L R R3
+L mows-rescue:R R3
 U 1 1 594FB633
 P 5050 1050
@@
 $EndComp
 $Comp
-L R R7
+L mows-rescue:R R7
 U 1 1 594FB669
 P 6100 1050
@@
 $EndComp
 $Comp
-L D_Schottky D1
+L mows-rescue:D_Schottky D1
 U 1 1 594FB69F
 P 3150 1250
@@
 $EndComp
 $Comp
-L GND #PWR01
+L mows-rescue:GND #PWR01
 U 1 1 594FC2C3
 P 5050 1700
@@
 Text Label 5350 1250 0    60   ~ 0
 VBATT
-Text Label 3350 950  0    60   ~ 0
-SUN
-$Comp
-L +3V3 #PWR02
+$Comp
+L mows-rescue:+3V3 #PWR02
 U 1 1 594FC5BB
 P 1750 1250
@@
 $EndComp
 $Comp
-L GND #PWR03
+L mows-rescue:GND #PWR03
 U 1 1 594FC61C
 P 2400 1650
@@
 SCK
 $Comp
-L +3V3 #PWR04
+L mows-rescue:+3V3 #PWR04
 U 1 1 594FD423
 P 4700 2400
@@
 $EndComp
 $Comp
-L GND #PWR05
+L mows-rescue:GND #PWR05
 U 1 1 594FD45E
 P 4700 2900
@@
 MOSI
 $Comp
-L +3V3 #PWR06
+L mows-rescue:+3V3 #PWR06
 U 1 1 594FF0D2
 P 1300 3450
@@
 $EndComp
 $Comp
-L GND #PWR07
+L mows-rescue:GND #PWR07
 U 1 1 594FF0F4
 P 1300 3950
@@
 RST
 $Comp
-L R R5
+L mows-rescue:R R5
 U 1 1 599B8E52
 P 5550 2250
@@
 $EndComp
 $Comp
-L R R6
+L mows-rescue:R R6
 U 1 1 599B9487
 P 5550 3350
@@
 RAIN
 $Comp
-L +3V3 #PWR08
+L mows-rescue:+3V3 #PWR08
 U 1 1 599B9EA3
 P 6100 850
@@
 $EndComp
 $Comp
-L GND #PWR09
+L mows-rescue:GND #PWR09
 U 1 1 599BA12B
 P 6100 1450
@@
 W_SPD
 $Comp
-L GND #PWR010
+L mows-rescue:GND #PWR010
 U 1 1 599BB276
 P 5550 2650
@@
 $EndComp
 $Comp
-L +3V3 #PWR011
+L mows-rescue:+3V3 #PWR011
 U 1 1 599BB3E3
 P 5550 2050
@@
 $EndComp
 $Comp
-L GND #PWR012
+L mows-rescue:GND #PWR012
 U 1 1 599BC73E
 P 5550 3750
@@
 W_DIR
 $Comp
-L +3V3 #PWR013
+L mows-rescue:+3V3 #PWR013
 U 1 1 599BCCE9
 P 5550 3150
@@
 DHT22
 $Comp
-L +3.3V #PWR014
+L mows-rescue:+3.3V #PWR014
 U 1 1 5A468922
 P 3950 3550
@@
 	1    0    0    -1
 $EndComp
-Text Label 3950 900  0    60   ~ 0
-SUN
-$Comp
-L GND #PWR015
+$Comp
+L mows-rescue:GND #PWR015
 U 1 1 5A46EB40
-P 4050 1650
-F 0 "#PWR015" H 4050 1400 50  0001 C CNN
-F 1 "GND" H 4050 1500 50  0000 C CNN
-F 2 "" H 4050 1650 50  0001 C CNN
-F 3 "" H 4050 1650 50  0001 C CNN
-	1    4050 1650
-	1    0    0    -1
-$EndComp
-$Comp
-L GND #PWR016
+P 3550 1650
+F 0 "#PWR015" H 3550 1400 50  0001 C CNN
+F 1 "GND" H 3550 1500 50  0000 C CNN
+F 2 "" H 3550 1650 50  0001 C CNN
+F 3 "" H 3550 1650 50  0001 C CNN
+	1    3550 1650
+	1    0    0    -1
+$EndComp
+$Comp
+L mows-rescue:GND #PWR016
 U 1 1 5A46EB72
-P 4050 1050
-F 0 "#PWR016" H 4050 800 50  0001 C CNN
-F 1 "GND" H 4050 900 50  0000 C CNN
-F 2 "" H 4050 1050 50  0001 C CNN
-F 3 "" H 4050 1050 50  0001 C CNN
-	1    4050 1050
-	1    0    0    -1
-$EndComp
-$Comp
-L GND #PWR017
+P 3550 1050
+F 0 "#PWR016" H 3550 800 50  0001 C CNN
+F 1 "GND" H 3550 900 50  0000 C CNN
+F 2 "" H 3550 1050 50  0001 C CNN
+F 3 "" H 3550 1050 50  0001 C CNN
+	1    3550 1050
+	1    0    0    -1
+$EndComp
+$Comp
+L mows-rescue:GND #PWR017
 U 1 1 5A472770
 P 4350 3800
@@
 $EndComp
 $Comp
-L Conn_01x02 con_sun1
+L mows-rescue:Conn_01x02 con_sun1
 U 1 1 5A47356F
-P 4350 900
-F 0 "con_sun1" H 4350 1000 50  0000 C CNN
-F 1 "SUN" H 4350 700 50  0000 C CNN
-F 2 "Pin_Headers:Pin_Header_Straight_1x02_Pitch2.54mm" H 4350 900 50  0001 C CNN
-F 3 "" H 4350 900 50  0001 C CNN
-	1    4350 900
-	1    0    0    -1
-$EndComp
-$Comp
-L Conn_01x02 con_bat1
+P 3850 900
+F 0 "con_sun1" H 3850 1000 50  0000 C CNN
+F 1 "SUN" H 3850 700 50  0000 C CNN
+F 2 "Pin_Headers:Pin_Header_Straight_1x02_Pitch2.54mm" H 3850 900 50  0001 C CNN
+F 3 "" H 3850 900 50  0001 C CNN
+	1    3850 900
+	1    0    0    -1
+$EndComp
+$Comp
+L mows-rescue:Conn_01x02 con_bat1
 U 1 1 5A4735FC
-P 4350 1500
-F 0 "con_bat1" H 4350 1600 50  0000 C CNN
-F 1 "BATT" H 4350 1300 50  0000 C CNN
-F 2 "Pin_Headers:Pin_Header_Straight_1x02_Pitch2.54mm" H 4350 1500 50  0001 C CNN
-F 3 "" H 4350 1500 50  0001 C CNN
-	1    4350 1500
-	1    0    0    -1
-$EndComp
-$Comp
-L Conn_01x03 J2
+P 3850 1500
+F 0 "con_bat1" H 3850 1600 50  0000 C CNN
+F 1 "BATT" H 3850 1300 50  0000 C CNN
+F 2 "Pin_Headers:Pin_Header_Straight_1x02_Pitch2.54mm" H 3850 1500 50  0001 C CNN
+F 3 "" H 3850 1500 50  0001 C CNN
+	1    3850 1500
+	1    0    0    -1
+$EndComp
+$Comp
+L mows-rescue:Conn_01x03 J2
 U 1 1 5A4740C8
 P 3200 3700
@@
 $EndComp
 $Comp
-L GND #PWR018
+L mows-rescue:GND #PWR018
 U 1 1 5A475913
 P 3000 3950
@@
 RFTX
 $Comp
-L +BATT #PWR019
-U 1 1 5A477DB3
-P 3000 1050
-F 0 "#PWR019" H 3000 900 50  0001 C CNN
-F 1 "+BATT" H 3000 1190 50  0000 C CNN
-F 2 "" H 3000 1050 50  0001 C CNN
-F 3 "" H 3000 1050 50  0001 C CNN
-	1    3000 1050
-	1    0    0    -1
-$EndComp
-$Comp
-L +BATT #PWR020
-U 1 1 5A478987
-P 3950 1500
-F 0 "#PWR020" H 3950 1350 50  0001 C CNN
-F 1 "+BATT" H 3950 1640 50  0000 C CNN
-F 2 "" H 3950 1500 50  0001 C CNN
-F 3 "" H 3950 1500 50  0001 C CNN
-	1    3950 1500
-	1    0    0    -1
-$EndComp
-$Comp
-L +BATT #PWR021
+L mows-rescue:+BATT #PWR021
 U 1 1 5A4793EE
 P 5050 850
@@
 $EndComp
 $Comp
-L Conn_01x06 J1
+L mows-rescue:Conn_01x06 J1
 U 1 1 5A467D4C
 P 1700 3650
@@
 $EndComp
 $Comp
-L R R1
+L mows-rescue:R R1
 U 1 1 5A469C7F
 P 2650 3750
@@
 $EndComp
 $Comp
-L R R2
+L mows-rescue:R R2
 U 1 1 5A46B1D0
 P 4050 3700
@@
 $EndComp
 $Comp
-L Conn_01x03 J3
+L mows-rescue:Conn_01x03 J3
 U 1 1 5A47AFD5
 P 4550 3650
@@
 $EndComp
 $Comp
-L Conn_01x02 J5
+L mows-rescue:Conn_01x02 J5
 U 1 1 5A47B11F
 P 5750 3600
@@
 $EndComp
 $Comp
-L Conn_01x02 J4
+L mows-rescue:Conn_01x02 J4
 U 1 1 5A47B19E
 P 5750 2500
@@
 $EndComp
 $Comp
-L Conn_01x02 J6
+L mows-rescue:Conn_01x02 J6
 U 1 1 5A47B467
 P 6300 1300
@@
 $EndComp
 $Comp
-L +BATT #PWR022
+L mows-rescue:+BATT #PWR022
 U 1 1 5A82E3BB
 P 2850 3800
@@
 	5550 3200 5550 3150
 Wire Wire Line
-	4150 900  3950 900
-Wire Wire Line
-	4150 1500 3950 1500
-Wire Wire Line
 	4350 3750 4350 3800
 Wire Wire Line
@@
 	2400 1550 2400 1650
 Wire Wire Line
-	4150 1600 4050 1600
-Wire Wire Line
-	4050 1600 4050 1650
-Wire Wire Line
-	4050 1050 4050 1000
-Wire Wire Line
-	4050 1000 4150 1000
+	3650 1600 3550 1600
+Wire Wire Line
+	3550 1600 3550 1650
+Wire Wire Line
+	3550 1050 3550 1000
+Wire Wire Line
+	3550 1000 3650 1000
 Wire Wire Line
 	5050 850  5050 900
@@
 	1750 1250 2100 1250
 $Comp
-L MCP1700-3302E_TO92 U1
+L mows-rescue:MCP1700-3302E_TO92 U1
 U 1 1 5A466099
 P 2400 1250
@@
 $EndComp
 Wire Wire Line
-	3350 950  3350 1250
-Wire Wire Line
 	3350 1250 3300 1250
 Wire Wire Line
-	3000 1050 3000 1250
-Wire Wire Line
-	3000 1250 2700 1250
+	3000 1250 2900 1250
+Wire Wire Line
+	2900 1500 2900 1250
+Connection ~ 2900 1250
+Wire Wire Line
+	2900 1250 2700 1250
+Wire Wire Line
+	3350 900  3350 1250
+Wire Wire Line
+	2900 1500 3650 1500
+Wire Wire Line
+	3650 900  3350 900
 $EndSCHEMATC
