File: hw/mows.sch (KiCad schematic (older format))
At the start: 18 parts, among them J1 Conn_01x05, J2 STX882, J3 DHT22, J4 WSPD, J5 WDIR, J6 RAIN, U1 MCP1700-3302E_TO92, U2 ATTINY85-20PU

Commit message: pcb labels
Parts:
- J1: footprint Connector_PinHeader_2.54mm:PinHeader_1x05_P2.54mm_Vertical -> Connector_PinSocket_2.54mm:PinSocket_1x05_P2.54mm_Vertical
Changed lines of the file:
@@
 F 0 "J1" H 1480 2242 50  0000 L CNN
 F 1 "Conn_01x05" H 1480 2151 50  0000 L CNN
-F 2 "Connector_PinHeader_2.54mm:PinHeader_1x05_P2.54mm_Vertical" H 1400 2200 50  0001 C CNN
+F 2 "Connector_PinSocket_2.54mm:PinSocket_1x05_P2.54mm_Vertical" H 1400 2200 50  0001 C CNN
 F 3 "~" H 1400 2200 50  0001 C CNN
 	1    1400 2200

Commit message: Some hardware commits
Parts:
- J1: symbol Connector_Generic:Conn_01x05 -> mows-rescue:Conn_01x05-Connector_Generic
Changed lines of the file:
@@
 EESchema Schematic File Version 4
-LIBS:mows-cache
 EELAYER 30 0
 EELAYER END
@@
 	950  1200 1250 1200
 $Comp
-L Connector_Generic:Conn_01x05 J1
+L mows-rescue:Conn_01x05-Connector_Generic J1
 U 1 1 5DB2544D
 P 1400 2200
