File: hw/mows.kicad_pcb (KiCad board)
At the start: 2 copper layers, 47 x 50.8 mm, 18 parts, among them J1 ICSP, J2 STX882, J3 DHT22, J4 WSPD, J5 WDIR, J6 RAIN, U1 MCP1700, U2 ATTINY85-20PU

Commit message: Nova placa
Parts:
- D1: value shottky -> D_Schottky
- J1: value ICSP -> Conn_01x05; footprint Pin_Headers:Pin_Header_Straight_1x06_Pitch2.54mm -> Connector_PinHeader_2.54mm:PinHeader_1x05_P2.54mm_Vertical
- J3: footprint Pin_Headers:Pin_Header_Straight_1x03_Pitch2.54mm -> Connector_PinHeader_2.54mm:PinHeader_1x03_P2.54mm_Horizontal
- J4, J5, J6, con_bat1, con_sun1: footprint Pin_Headers:Pin_Header_Straight_1x02_Pitch2.54mm -> Connector_PinHeader_2.54mm:PinHeader_1x02_P2.54mm_Horizontal
- U1: value MCP1700 -> MCP1700-3302E_TO92
- moved con_sun1 22.6 mm to (150.8, 75.2), turned to 0 degrees
- moved J3 16.1 mm to (147.2, 109.0), turned to 270 degrees
- moved J5 15.2 mm to (166.0, 109.0), turned to 270 degrees
- moved R2 11.1 mm to (167.1, 102.1)
- moved J6 10.3 mm to (153.5, 109.0), turned to 270 degrees
- moved D1 9.27 mm to (134.0, 75.2), turned to 0 degrees
- moved con_bat1 8.62 mm to (150.9, 81.9), turned to 0 degrees
- moved J4 8.45 mm to (159.8, 109.0), turned to 270 degrees
- moved R7 7.81 mm to (167.1, 97.8)
- moved R5 4.42 mm to (167.1, 93.7)
- moved R3 4.17 mm to (136.9, 84.2)
- moved J1 2.07 mm to (153.9, 89.7)
- moved U1 1.93 mm to (145.5, 80.7)
- moved R6 1.79 mm to (167.1, 89.9)
- moved R4 1.60 mm to (136.9, 88.4)
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Connections:
- net /SUN renamed Net-(D1-Pad2)
- J1 pad 1: +3V3 -> /RST
- J1 pad 2: /RST -> /SCK
- J1 pad 3: /SCK -> /MISO
- J1 pad 4: /MISO -> /MOSI
- J1 pad 5: /MOSI -> GND
- U1 pad 2: +3V3 -> +BATT
- U1 pad 3: +BATT -> +3V3
Routing:
- net GND: track 141.3 -> 0.00 mm
- net +3V3: track 91.1 -> 65.7 mm
- net /SCK: track 21.7 -> 38.1 mm
- net /MISO: track 21.7 -> 34.1 mm
- net /DHT22: track 35.0 -> 30.6 mm
- net /RST: track 27.5 -> 31.5 mm
Other:
- board size 47 x 50.8 mm -> 48 x 60 mm
- board text added: "+"
- board text added: "-"
- board text added: "DATA"
- board text added: "GND"
- board text added: "MISO"
- board text added: "MOSI"
- board text added: "MOWS station v1910"
- board text added: "RST"
- board text added: "SCK"
- board text added: "VBAT"

Commit message: pcb labels
Parts:
- J1: footprint Connector_PinHeader_2.54mm:PinHeader_1x05_P2.54mm_Vertical -> Connector_PinSocket_2.54mm:PinSocket_1x05_P2.54mm_Vertical
Changed lines of the file:
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@@
-    )
-  )
-  (module Connector_PinHeader_2.54mm:PinHeader_1x05_P2.54mm_Vertical (layer F.Cu)
-    (at 153.9 89.69)
-    (descr "Through hole straight pin header, 1x05, 2.54mm pitch, single row")
-    (tags "Through hole pin header THT 1x05 2.54mm single row")
-    (fp_text reference J1 (at 0 -2.33) (layer F.SilkS)
-      (effects (font (size 1 1) (thickness 0.15)))
-    )
-    (fp_text value Conn_01x05 (at 0 12.49) (layer F.Fab)
-      (effects (font (size 1 1) (thickness 0.15)))
-    )
-    (fp_text user %R (at 0 5.08 90) (layer F.Fab)
-      (effects (font (size 1 1) (thickness 0.15)))
-    )
-    (fp_line (start 1.8 -1.8) (end -1.8 -1.8) (layer F.CrtYd) (width 0.05))
-    (fp_line (start 1.8 11.95) (end 1.8 -1.8) (layer F.CrtYd) (width 0.05))
-    (fp_line (start -1.8 11.95) (end 1.8 11.95) (layer F.CrtYd) (width 0.05))
-    (fp_line (start -1.8 -1.8) (end -1.8 11.95) (layer F.CrtYd) (width 0.05))
-    (fp_line (start -1.33 -1.33) (end 0 -1.33) (layer F.SilkS) (width 0.12))
-    (fp_line (start -1.33 0) (end -1.33 -1.33) (layer F.SilkS) (width 0.12))
-    (fp_line (start -1.33 1.27) (end 1.33 1.27) (layer F.SilkS) (width 0.12))
-    (fp_line (start 1.33 1.27) (end 1.33 11.49) (layer F.SilkS) (width 0.12))
-    (fp_line (start -1.33 1.27) (end -1.33 11.49) (layer F.SilkS) (width 0.12))
-    (fp_line (start -1.33 11.49) (end 1.33 11.49) (layer F.SilkS) (width 0.12))
-    (fp_line (start -1.27 -0.635) (end -0.635 -1.27) (layer F.Fab) (width 0.1))
-    (fp_line (start -1.27 11.43) (end -1.27 -0.635) (layer F.Fab) (width 0.1))
-    (fp_line (start 1.27 11.43) (end -1.27 11.43) (layer F.Fab) (width 0.1))
-    (fp_line (start 1.27 -1.27) (end 1.27 11.43) (layer F.Fab) (width 0.1))
-    (fp_line (start -0.635 -1.27) (end 1.27 -1.27) (layer F.Fab) (width 0.1))
-    (pad 5 thru_hole oval (at 0 10.16) (size 1.7 1.7) (drill 1) (layers *.Cu *.Mask)
-      (net 2 GND))
-    (pad 4 thru_hole oval (at 0 7.62) (size 1.7 1.7) (drill 1) (layers *.Cu *.Mask)
-      (net 5 /MOSI))
-    (pad 3 thru_hole oval (at 0 5.08) (size 1.7 1.7) (drill 1) (layers *.Cu *.Mask)
-      (net 8 /MISO))
-    (pad 2 thru_hole oval (at 0 2.54) (size 1.7 1.7) (drill 1) (layers *.Cu *.Mask)
-      (net 7 /SCK))
-    (pad 1 thru_hole rect (at 0 0) (size 1.7 1.7) (drill 1) (layers *.Cu *.Mask)
-      (net 9 /RST))
-    (model ${KISYS3DMOD}/Connector_PinHeader_2.54mm.3dshapes/PinHeader_1x05_P2.54mm_Vertical.wrl
-      (at (xyz 0 0 0))
-      (scale (xyz 1 1 1))
-      (rotate (xyz 0 0 0))
     )
   )
@@
     )
   )
+  (module Connector_PinSocket_2.54mm:PinSocket_1x05_P2.54mm_Vertical (layer F.Cu)
+    (at 153.9 89.69)
+    (descr "Through hole straight socket strip, 1x05, 2.54mm pitch, single row (from Kicad 4.0.7), script generated")
+    (tags "Through hole socket strip THT 1x05 2.54mm single row")
+    (fp_text reference J1 (at 0 -2.77) (layer F.SilkS)
+      (effects (font (size 1 1) (thickness 0.15)))
+    )
+    (fp_text value Conn_01x05 (at 0 12.93) (layer F.Fab)
+      (effects (font (size 1 1) (thickness 0.15)))
+    )
+    (fp_line (start -1.27 -1.27) (end 0.635 -1.27) (layer F.Fab) (width 0.1))
+    (fp_line (start 0.635 -1.27) (end 1.27 -0.635) (layer F.Fab) (width 0.1))
+    (fp_line (start 1.27 -0.635) (end 1.27 11.43) (layer F.Fab) (width 0.1))
+    (fp_line (start 1.27 11.43) (end -1.27 11.43) (layer F.Fab) (width 0.1))
+    (fp_line (start -1.27 11.43) (end -1.27 -1.27) (layer F.Fab) (width 0.1))
+    (fp_line (start -1.33 1.27) (end 1.33 1.27) (layer F.SilkS) (width 0.12))
+    (fp_line (start -1.33 1.27) (end -1.33 11.49) (layer F.SilkS) (width 0.12))
+    (fp_line (start -1.33 11.49) (end 1.33 11.49) (layer F.SilkS) (width 0.12))
+    (fp_line (start 1.33 1.27) (end 1.33 11.49) (layer F.SilkS) (width 0.12))
+    (fp_line (start 1.33 -1.33) (end 1.33 0) (layer F.SilkS) (width 0.12))
+    (fp_line (start 0 -1.33) (end 1.33 -1.33) (layer F.SilkS) (width 0.12))
+    (fp_line (start -1.8 -1.8) (end 1.75 -1.8) (layer F.CrtYd) (width 0.05))
+    (fp_line (start 1.75 -1.8) (end 1.75 11.9) (layer F.CrtYd) (width 0.05))
+    (fp_line (start 1.75 11.9) (end -1.8 11.9) (layer F.CrtYd) (width 0.05))
+    (fp_line (start -1.8 11.9) (end -1.8 -1.8) (layer F.CrtYd) (width 0.05))
+    (fp_text user %R (at 0 5.08 90) (layer F.Fab)
+      (effects (font (size 1 1) (thickness 0.15)))
+    )
+    (pad 1 thru_hole rect (at 0 0) (size 1.7 1.7) (drill 1) (layers *.Cu *.Mask)
+      (net 9 /RST))
+    (pad 2 thru_hole oval (at 0 2.54) (size 1.7 1.7) (drill 1) (layers *.Cu *.Mask)
+      (net 7 /SCK))
+    (pad 3 thru_hole oval (at 0 5.08) (size 1.7 1.7) (drill 1) (layers *.Cu *.Mask)
+      (net 8 /MISO))
+    (pad 4 thru_hole oval (at 0 7.62) (size 1.7 1.7) (drill 1) (layers *.Cu *.Mask)
+      (net 5 /MOSI))
+    (pad 5 thru_hole oval (at 0 10.16) (size 1.7 1.7) (drill 1) (layers *.Cu *.Mask)
+      (net 2 GND))
+    (model ${KISYS3DMOD}/Connector_PinSocket_2.54mm.3dshapes/PinSocket_1x05_P2.54mm_Vertical.wrl
+      (at (xyz 0 0 0))
+      (scale (xyz 1 1 1))
+      (rotate (xyz 0 0 0))
+    )
+  )
   (gr_text "MOWS station v1910" (at 147 71.25) (layer F.SilkS)
     (effects (font (size 1.2 1.2) (thickness 0.2)))
@@
   (segment (start 135.75063 84.25) (end 133.104 86.89663) (width 0.5) (layer F.Cu) (net 1))
   (segment (start 136.882 84.25) (end 135.75063 84.25) (width 0.5) (layer F.Cu) (net 1) (status 10))
+  (segment (start 150.8139 82.0065) (end 150.87232 81.94808) (width 0.5) (layer F.Cu) (net 1) (status 30))
+  (segment (start 145.4545 82.0065) (end 150.8139 82.0065) (width 0.5) (layer F.Cu) (net 1) (status 30))
+  (segment (start 139.1555 82.0065) (end 133.961 76.812) (width 0.5) (layer F.Cu) (net 1))
+  (segment (start 145.4545 82.0065) (end 139.1555 82.0065) (width 0.5) (layer F.Cu) (net 1) (status 10))
+  (segment (start 133.961 76.812) (end 133.961 75.212) (width 0.5) (layer F.Cu) (net 1) (status 20))
+  (segment (start 137.711999 83.450001) (end 139.1555 82.0065) (width 0.5) (layer F.Cu) (net 1))
+  (segment (start 137.681999 83.450001) (end 137.711999 83.450001) (width 0.5) (layer F.Cu) (net 1))
+  (segment (start 136.882 84.25) (end 137.681999 83.450001) (width 0.5) (layer F.Cu) (net 1) (status 10))
   (segment (start 139.31537 97.294) (end 146.058 104.03663) (width 0.5) (layer B.Cu) (net 3))
   (segment (start 138.184 97.294) (end 139.31537 97.294) (width 0.5) (layer B.Cu) (net 3) (status 10))
@@
   (segment (start 133.416 88.404) (end 136.914 88.404) (width 0.5) (layer B.Cu) (net 9) (status 20))
   (segment (start 129.262 84.25) (end 133.416 88.404) (width 0.5) (layer B.Cu) (net 9) (status 10))
-  (segment (start 150.8139 82.0065) (end 150.87232 81.94808) (width 0.5) (layer F.Cu) (net 1) (status 30))
-  (segment (start 145.4545 82.0065) (end 150.8139 82.0065) (width 0.5) (layer F.Cu) (net 1) (status 30))
-  (segment (start 139.1555 82.0065) (end 133.961 76.812) (width 0.5) (layer F.Cu) (net 1))
-  (segment (start 145.4545 82.0065) (end 139.1555 82.0065) (width 0.5) (layer F.Cu) (net 1) (status 10))
-  (segment (start 133.961 76.812) (end 133.961 75.212) (width 0.5) (layer F.Cu) (net 1) (status 20))
-  (segment (start 137.711999 83.450001) (end 139.1555 82.0065) (width 0.5) (layer F.Cu) (net 1))
-  (segment (start 137.681999 83.450001) (end 137.711999 83.450001) (width 0.5) (layer F.Cu) (net 1))
-  (segment (start 136.882 84.25) (end 137.681999 83.450001) (width 0.5) (layer F.Cu) (net 1))
   (segment (start 150.77072 75.212) (end 150.8012 75.18152) (width 0.5) (layer F.Cu) (net 10) (status 30))
   (segment (start 146.661 75.212) (end 150.77072 75.212) (width 0.5) (layer F.Cu) (net 10) (status 30))
